Commit message: urdf cleaner

File: src/robotic_arm/urdf/robotic_arm.urdf (robot description, URDF)
Before this commit: robot robotic_arm, 6 links, 5 joints
Links:
- link base_link: mass None -> 0.001

Commit message: addition of corrected models

File: src/robotic_arm/urdf/robotic_arm.urdf (robot description, URDF)
Before this commit: robot robotic_arm, 6 links, 5 joints
Links:
- added link world
- link arm_base: geometry collision mesh filename=package://robotic_arm/gazebo_models/collision/arm_base_coll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; visual mesh filename=package://robotic_arm/gazebo_models/visual/arm_base.stl
- link arm_link_1: geometry collision mesh filename=package://robotic_arm/gazebo_models/collision/arm_link_1_co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; visual mesh filename=package://robotic_arm/gazebo_models/visual/arm_link_1.stl
- link arm_link_2: geometry collision mesh filename=package://robotic_arm/gazebo_models/collision/arm_link_2_co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; visual mesh filename=package://robotic_arm/gazebo_models/visual/arm_link_2.stl
- link base_link: geometry collision box size=0.5 0.2 0.001; visual mesh filename=package://robotic_arm/meshes/base_link.STL
- link capstan_drive: geometry collision mesh filename=package://robotic_arm/gazebo_models/collision/capstan_colli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; visual mesh filename=package://robotic_arm/gazebo_models/visual/capstan_drive.stl
Joints:
- added joint base_link_fixed: type fixed, parent world, child base_link, origin xyz=0 0 0 rpy=0 0 0
- joint arm_elbow: origin xyz=4.1173E-05 0.005238 0.1 rpy=0.0068467 -0.00071181 0 -> xyz=4.1173E-05 0.005238 0.125 rpy=0.0068467 -0.00071181 0

Commit message: work out collisions make them smaller

File: src/robotic_arm/urdf/robotic_arm.urdf (robot description, URDF)
Before this commit: robot robotic_arm, 7 links, 6 joints
Links:
- link arm_base: geometry collision mesh filename=package://robotic_arm/gazebo_models/collision/arm_base_coll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; visual mesh filename=package://robotic_arm/meshes/arm_base.STL
- link arm_link_1: geometry collision mesh filename=package://robotic_arm/gazebo_models/collision/arm_link_1_co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; visual mesh filename=package://robotic_arm/meshes/arm_link_1.STL
- link arm_link_2: geometry collision mesh filename=package://robotic_arm/gazebo_models/collision/arm_link_2_co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; visual mesh filename=package://robotic_arm/meshes/arm_link_2.STL
- link capstan_drive: geometry collision mesh filename=package://robotic_arm/gazebo_models/collision/capstan_colli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; visual mesh filename=package://robotic_arm/meshes/capstan_drive.STL

Commit message: pid configured for arm

File: src/robotic_arm/urdf/robotic_arm.urdf (robot description, URDF)
Before this commit: robot robotic_arm, 7 links, 6 joints
Links:
- link arm_base: geometry visual mesh filename=package://robotic_arm/meshes/arm_base.STL
- link arm_link_1: geometry visual mesh filename=package://robotic_arm/meshes/arm_link_1.STL
- link arm_link_2: geometry visual mesh filename=package://robotic_arm/meshes/arm_link_2.STL
- link base_link: geometry visual mesh filename=package://robotic_arm/meshes/base_link.STL
- link capstan_drive: geometry visual mesh filename=package://robotic_arm/meshes/capstan_drive.STL

Commit message: finalised work

File: src/robotic_arm/urdf/robotic_arm.urdf (robot description, URDF)
Before this commit: robot robotic_arm, 7 links, 6 joints
Links:
- link base_link: geometry collision box size=0.5 0.2 0.001; visual mesh filename=package://robotic_arm/meshes/base_link.STL
